File: 电路/主控器/PM_Controller/PM_Controller.kicad_pcb (KiCad board)
At the start: 4 copper layers, 90 x 61.5 mm, 134 parts, among them J1 Conn_01x04_Socket, J10 Conn_02x04_Odd_Even, J11 Conn_02x06_Odd_Even, J2 Conn_01x04_Socket, J3 Conn_01x04_Socket, J4 Conn_01x04_Socket, J5 Conn_01x02_Pin, J6 Conn_01x02_Pin, J7 Conn_02x04_Odd_Even, J8 Conn_01x04_Pin, J9 Conn_01x04_Socket, P2V5 SolderJumper_2_Open, P3V3 SolderJumper_2_Open, Q1 AO3401A, Q2 AO3400A, Q3 AO3400A, Q4 AO3400A, Q5 AO3400A, Q6 AO3400A, U1 AT24CS08-SSHM, U10 TMP102xxDRL, U11 TPS2552DDBVR, U12 TLP127, U2 AMS1117-3.3, U3 STM32G431RBTx, U4 TPS61085DGK, U5 BQ21040DBV, U6 TPS2552DDBVR, U7 STM32L011D4Px, U8 ME6211C25M5, U9 AT24CS08-SSHM, Y1 32.768kHz, Y2 24Mhz

Commit message: ZUI init
Parts:
- removed C13: 22uf, Capacitor_SMD:C_0603_1608Metric_Pad1.08x0.95mm_HandSolder
- removed C15: 100nf, Capacitor_SMD:C_0603_1608Metric_Pad1.08x0.95mm_HandSolder
- removed C16: 820pf, Capacitor_SMD:C_0603_1608Metric_Pad1.08x0.95mm_HandSolder
- removed C4: 22uf, Capacitor_Tantalum_SMD:CP_EIA-3528-21_Kemet-B_Pad1.50x2.35mm_HandSolder
- removed C9: 1uf, Capacitor_SMD:C_0603_1608Metric_Pad1.08x0.95mm_HandSolder
- removed D1: SS32, Diode_SMD:D_SMA_Handsoldering
- removed R10: 82k, Resistor_SMD:R_0603_1608Metric_Pad0.98x0.95mm_HandSolder
- removed R11: 27k, Resistor_SMD:R_0603_1608Metric_Pad0.98x0.95mm_HandSolder
- removed R9: 56.2k, Resistor_SMD:R_0603_1608Metric_Pad0.98x0.95mm_HandSolder
- removed U4: TPS61085DGK, Package_SO:VSSOP-8_3x3mm_P0.65mm
- added C39: 22uf, Capacitor_Tantalum_SMD:CP_EIA-3528-21_Kemet-B_HandSolder, F.Cu at (62.8, 154.8)
- added C40: 1uf, Capacitor_SMD:C_1206_3216Metric_Pad1.33x1.80mm_HandSolder, F.Cu at (57.3, 144.2)
- added C41: 10uf, Capacitor_SMD:C_1206_3216Metric_Pad1.33x1.80mm_HandSolder, F.Cu at (59.1, 155.7)
- added D4: 1N5819WS, Diode_SMD:D_SOD-323_HandSoldering, F.Cu at (56.3, 155.5)
- added R43: 330k, Resistor_SMD:R_0603_1608Metric_Pad0.98x0.95mm_HandSolder, F.Cu at (63.9, 149.9)
- added R44: 51k, Resistor_SMD:R_0603_1608Metric_Pad0.98x0.95mm_HandSolder, F.Cu at (63.9, 148.4)
- added R45: 10k, Resistor_SMD:R_0603_1608Metric_Pad0.98x0.95mm_HandSolder, F.Cu at (61.1, 146.4)
- added U13: TLV61048DBVR, footprints:SOT-23-6_DBV_TEX, F.Cu at (59.1, 149.6)
- J5: footprint Connector_Wire:SolderWire-0.1sqmm_1x02_P3.6mm_D0.4mm_OD1mm_Relief -> Connector_Wire:SolderWire-0.5sqmm_1x02_P4.8mm_D0.9mm_OD2.3mm
- L1: footprint Inductor_SMD:L_APV_ANR5040 -> Inductor_SMD:L_APV_APH0650
- moved L1 7.21 mm to (51.4, 150.2), turned to -90 degrees
- moved J5 6.00 mm to (54.1, 137.2), turned to 0 degrees
- moved R25 2.21 mm to (68.5, 145.2)
- moved C11 1.17 mm to (58.6, 156.1)
- moved R23 0.45 mm to (62.5, 142.5), turned to -90 degrees
- moved R24 0.45 mm to (64.0, 142.5)
- moved C6 0.15 mm to (66.9, 160.1)
Routing:
- net /BAT_OUT: track 28.0 -> 5.81 mm, vias 2 -> 5
- net Net-(U13-FB): track 0.00 -> 5.83 mm
- net Net-(U4-FB): track 5.30 -> 0.00 mm, vias 1 -> 0
- net Net-(D4-A): track 6.27 -> 1.46 mm
- net Net-(U4-SS): track 4.29 -> 0.00 mm
- net /VBAT5: track 7.26 -> 3.78 mm, vias 1 -> 0
- net Net-(U13-EN): track 0.00 -> 3.23 mm
- net Net-(C16-Pad2): track 2.40 -> 0.00 mm
- net /ADC1_15: track 34.2 -> 31.9 mm
- net Net-(U4-COMP): track 1.77 -> 0.00 mm
- net Net-(R23-Pad1): track 5.63 -> 7.22 mm
- net GND: track 101.2 -> 101.7 mm, vias 100 -> 102
- net +BATT: vias 10 -> 9
- removed copper zone on F.Cu, net Net-(U4-SS)
Other:
- outline, holes or cut-outs redrawn

Commit message: 闪光灯ok
Parts:
- removed P2V5: SolderJumper_2_Open, Jumper:SolderJumper-2_P1.3mm_Open_RoundedPad1.0x1.5mm
- added L2: 4.7uH, Inductor_SMD:L_APV_APH0650, F.Cu at (86.5, 153.6)
- added L3: 4.7uH, Inductor_SMD:L_APV_APH0650, F.Cu at (68.6, 131.1)
- C24, C38: moved to B.Cu
- R43: value 330k -> 150k
- R44: value 51k -> 33k
- moved C24 12.2 mm to (98.3, 157.5), turned to -90 degrees
- moved C17 4.74 mm to (94.3, 156.6), turned to 0 degrees
- moved C38 2.55 mm to (69.9, 136.1), turned to 0 degrees
- moved C8 1.25 mm to (66.1, 162.6)
- moved C6 0.65 mm to (66.2, 160.1)
- moved J3 0.60 mm to (86.1, 159.1)
- moved C18 0.54 mm to (91.7, 149.8)
- moved R8 0.19 mm to (69.1, 156.5)
Connections:
- C17 pad 1: +5V -> Net-(U2-VI)
- J3 pad 1: Net-(J3-Pin_1) -> unconnected-(J3-Pin_1-Pad1)
- J9 pad 1: /BAT_OUT2 -> Net-(J9-Pin_1)
- U2 pad 3: +5V -> Net-(U2-VI)
Routing:
- net GND: track 101.7 -> 108.6 mm, vias 102 -> 103
- net Net-(J9-Pin_1): track 0.00 -> 4.32 mm
- net Net-(J3-Pin_1): track 3.22 -> 0.00 mm
- net /BAT_OUT2: track 0.00 -> 1.35 mm, vias 0 -> 1
- net +2V5: track 19.0 -> 17.7 mm, vias 1 -> 0
- net /EJCMT_EN: track 34.6 -> 35.8 mm
- net +5VA: track 28.5 -> 29.7 mm
- net +BATT: track 14.0 -> 14.4 mm, vias 9 -> 21
- net +3.3V: vias 25 -> 27
- added copper zone on In2.Cu, net +BATT
- added copper zone on F.Cu, net Net-(U2-VI)

Commit message: 优化外壳与5V外部供电电路选择逻辑
Parts:
- removed D2: SS32, Diode_SMD:D_SMA_Handsoldering
- removed Q1: AO3401A, Package_TO_SOT_SMD:SOT-23
- removed Q4: AO3400A, Package_TO_SOT_SMD:SOT-23
- removed R19: 100k, Resistor_SMD:R_0603_1608Metric_Pad0.98x0.95mm_HandSolder
- added C4: 100nf, Capacitor_SMD:C_0603_1608Metric, F.Cu at (65.8, 150.3)
- added D1: SS34, Diode_SMD:D_SMA, F.Cu at (88.7, 158.8)
- added H9: MountingHole_Pad, MountingHole:MountingHole_3.2mm_M3_DIN965_Pad_TopBottom, F.Cu at (59.5, 139.5)
- C12: value 47uf -> 22uf; footprint Capacitor_Tantalum_SMD:CP_EIA-3528-21_Kemet-B_Pad1.50x2.35mm_HandSolder -> Capacitor_SMD:C_1206_3216Metric_Pad1.33x1.80mm_HandSolder
- C35, R3: moved to B.Cu
- R25, R26, R32, R40: value 100k -> 1k
- R6: value 100k -> 1k; moved to B.Cu
- R7: moved to F.Cu
- moved CHG1 59.4 mm to (119.0, 157.0), turned to 180 degrees
- moved PW_LED1 56.9 mm to (119.0, 158.9), turned to 180 degrees
- moved C12 42.9 mm to (65.0, 120.6), turned to 180 degrees
- moved C5 31.5 mm to (97.8, 159.9), turned to 90 degrees
- moved R6 30.9 mm to (66.2, 133.4), turned to -135 degrees
- moved J3 27.3 mm to (62.4, 172.7)
- moved R3 19.0 mm to (82.9, 162.3), turned to 90 degrees
- moved U10 17.6 mm to (128.9, 158.8)
- moved R7 17.3 mm to (79.5, 158.9)
- moved C36 17.1 mm to (129.1, 155.5)
- moved C10 16.2 mm to (83.3, 162.3), turned to -90 degrees
- moved U5 11.8 mm to (79.7, 162.8), turned to 0 degrees
- moved C8 10.2 mm to (76.3, 161.7), turned to 90 degrees
- moved R27 7.73 mm to (119.7, 148.6), turned to 180 degrees
- moved R4 7.47 mm to (71.2, 169.0), turned to 90 degrees
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Connections:
- C12 pad 1: +5VA -> +3.3V
- C39 pad 1: /VBAT5 -> +5V
- C41 pad 1: /VBAT5 -> +5V
- D4 pad 1: /VBAT5 -> +5V
- J5 pad 1: +BATT -> Net-(J5-Pin_1)
- J5 pad 2: /EJCMT_GND -> GND
- R43 pad 1: /VBAT5 -> +5V
- R6 pad 1: GND -> /EJCMT_EN
- R6 pad 2: +5VA -> Net-(J5-Pin_1)
Routing:
- net Net-(CHG1-A): track 6.69 -> 52.2 mm, vias 0 -> 2
- net /PWR_LED: track 22.2 -> 53.8 mm, vias 1 -> 2
- net /#CHRG: track 15.5 -> 45.6 mm, vias 0 -> 2
- net GND: track 108.6 -> 131.2 mm, vias 103 -> 100
- net Net-(PW_LED1-A): track 22.3 -> 41.7 mm, vias 1 -> 2
- net Net-(J5-Pin_1): track 0.00 -> 12.6 mm
- net /I2C2_SDA: track 45.8 -> 58.1 mm, vias 3 -> 4
- net /I2C2_SCL: track 46.3 -> 57.9 mm, vias 3 -> 4
- net +BATT: track 14.4 -> 25.7 mm, vias 21 -> 14
- net /SWDIO0: track 12.9 -> 23.8 mm
- net /WKUP: track 23.8 -> 15.8 mm
- net +5VA: track 29.7 -> 22.3 mm
- net /EJCMT_EN: track 35.8 -> 30.1 mm
- net /SWCLK0: track 16.5 -> 21.8 mm
- net Net-(R23-Pad1): track 7.22 -> 3.00 mm
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- removed copper zone on B.Cu, net /EJCMT_GND
- removed copper zone on F.Cu, net /VBAT5
Other:
- outline, holes or cut-outs redrawn
- board text added: "EN+"
- board text added: "GND"

Commit message: 主控升级至Rev1.2，电机驱动 Rev1.1
电机驱动修改后采用Mosfet控制高侧电源通路。主控配套进行了更改。
Parts:
- added C1: 10uf, Capacitor_SMD:C_1206_3216Metric_Pad1.33x1.80mm_HandSolder, F.Cu at (95.5, 99.2)
- added C2: 1uf, Capacitor_SMD:C_1206_3216Metric_Pad1.33x1.80mm_HandSolder, F.Cu at (106.8, 99.7)
- added C4: 100uf, Capacitor_SMD:CP_Elec_6.3x7.7, F.Cu at (112.5, 98.0)
- added D1: 1N5819WS, Diode_SMD:D_SOD-323_HandSoldering, F.Cu at (95.0, 96.7)
- added D3: LED, LED_SMD:LED_0805_2012Metric_Pad1.15x1.40mm_HandSolder, F.Cu at (123.0, 85.7)
- added D4: 1N5819WS, Diode_SMD:D_SOD-323_HandSoldering, F.Cu at (93.5, 93.2)
- added FB1: FerriteBead, Inductor_SMD:L_0603_1608Metric, B.Cu at (124.1, 94.5)
- added H1: MountingHole, MountingHole:MountingHole_3.2mm_M3, F.Cu at (116.0, 80.7)
- added H2: MountingHole, MountingHole:MountingHole_3.2mm_M3, F.Cu at (116.0, 105.7)
- added H4: MountingHole, MountingHole:MountingHole_3.2mm_M3, F.Cu at (85.0, 105.7)
- added J1: Conn_01x04_MountingPin, Connector_JST:JST_PH_S4B-PH-SM4-TB_1x04-1MP_P2.00mm_Horizontal, F.Cu at (122.7, 94.5)
- added J2: Conn_01x02_MountingPin, Connector_JST:JST_PH_S2B-PH-SM4-TB_1x02-1MP_P2.00mm_Horizontal, F.Cu at (86.0, 96.7)
- added L2: 4.7uH, Inductor_SMD:L_APV_APH1265, F.Cu at (102.5, 87.7)
- added Q1: AO3400A, Package_TO_SOT_SMD:SOT-23, B.Cu at (115.5, 98.4)
- added R1: 330k, Resistor_SMD:R_0603_1608Metric_Pad0.98x0.95mm_HandSolder, F.Cu at (100.0, 101.7)
- added R2: 51k, Resistor_SMD:R_0603_1608Metric_Pad0.98x0.95mm_HandSolder, F.Cu at (103.0, 104.2)
- added R4: 10k, Resistor_SMD:R_0603_1608Metric_Pad0.98x0.95mm_HandSolder, F.Cu at (116.6, 87.0)
- added R5: 1k, Resistor_SMD:R_0603_1608Metric, F.Cu at (113.8, 92.6)
- added U1: TLV61048DBVR, footprints:SOT-23-6_DBV_TEX, F.Cu at (102.7, 99.1)
Routing:
- net +BATT: track 25.7 -> 49.2 mm
- net /Motor+: track 0.00 -> 19.3 mm
- net GND: track 131.2 -> 148.5 mm, vias 100 -> 141
- net Net-(U1-EN): track 0.00 -> 15.9 mm
- net /POWER_GND: track 0.00 -> 6.35 mm, vias 0 -> 8
- net /SW: track 0.00 -> 5.20 mm
- net Net-(U1-FB): track 0.00 -> 5.17 mm
- net Net-(D3-A): track 0.00 -> 5.00 mm
- net /MT_EN: track 0.00 -> 4.97 mm, vias 0 -> 1
- net Net-(J1-Pin_3): track 0.00 -> 4.31 mm, vias 0 -> 1
- net (no net): vias 0 -> 8
- added copper zone on F.Cu, net /Motor+
- added copper zone on B.Cu, net /POWER_GND
- added copper zone on F.Cu, net /POWER_GND
- added copper zone on F.Cu, net /SW
- added copper zone on In2.Cu, net GND
Other:
- board size 90 x 61.5 mm -> 90 x 98.3 mm
- board text added: "12mm"
- board text added: "13.5mm"
- board text added: "13mm"
- board text added: "25mm"
- board text added: "31mm"
- board text added: "33mm"
- board text added: "5mm"
- board text added: "Controller For PM1"
- board text added: "Motor Driver For PM1"
- board text added: "R2.5"
- board text added: "Rev1.1"
- board text added: "Rev1.2"

Commit message: 更新了电机驱动以及主控器PCB
Parts:
- removed the C1 at (95.5, 99.2)
- removed the C2 at (106.8, 99.7)
- removed the C4 at (112.5, 98.0)
- removed the D1 at (95.0, 96.7)
- removed the D3 at (123.0, 85.7)
- removed the D4 at (93.5, 93.2)
- removed the FB1 at (124.1, 94.5)
- removed the H1 at (116.0, 80.7)
- removed the H2 at (116.0, 105.7)
- removed the H4 at (85.0, 105.7)
- removed the J1 at (122.7, 94.5)
- removed the J2 at (86.0, 96.7)
- removed the L2 at (102.5, 87.7)
- removed Q1: AO3400A, Package_TO_SOT_SMD:SOT-23
- removed the R1 at (100.0, 101.7)
- removed the R2 at (103.0, 104.2)
- removed the R4 at (116.6, 87.0)
- removed the R5 at (113.8, 92.6)
- removed the U1 at (102.7, 99.1)
Routing:
- net +BATT: track 49.2 -> 25.7 mm
- net /Motor+: track 19.3 -> 0.00 mm
- net GND: track 148.5 -> 131.2 mm, vias 141 -> 100
- net Net-(U1-EN): track 15.9 -> 0.00 mm
- net /POWER_GND: track 6.35 -> 0.00 mm, vias 8 -> 0
- net /SW: track 5.20 -> 0.00 mm
- net Net-(U1-FB): track 5.17 -> 0.00 mm
- net Net-(D3-A): track 5.00 -> 0.00 mm
- net /MT_EN: track 4.97 -> 0.00 mm, vias 1 -> 0
- net Net-(J1-Pin_3): track 4.31 -> 0.00 mm, vias 1 -> 0
- net (no net): vias 8 -> 0
- removed copper zone on F.Cu, net /Motor+
- removed copper zone on B.Cu, net /POWER_GND
- removed copper zone on F.Cu, net /POWER_GND
- removed copper zone on F.Cu, net /SW
- removed copper zone on In2.Cu, net GND
Other:
- board size 90 x 98.3 mm -> 90 x 61.5 mm
- board text removed: "12mm"
- board text removed: "13.5mm"
- board text removed: "13mm"
- board text removed: "25mm"
- board text removed: "31mm"
- board text removed: "33mm"
- board text removed: "5mm"
- board text removed: "Motor Driver For PM1"
- board text removed: "R2.5"
- board text removed: "Rev1.1"

Commit message: 硬件1.3版本，调整闪光灯为默认过MCU
Parts:
- turned JP1 to 180 degrees
Connections:
- JP1 pad 1: /SHUT_Trig+ -> /_FLASH_Trig_
- JP1 pad 3: /_FLASH_Trig_ -> /SHUT_Trig+
Changed lines of the file:
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@@
 	(title_block
 		(title "PM Controller")
-		(date "2026-01-21")
-		(rev "1.2")
+		(date "2026-02-03")
+		(rev "1.3")
 		(company "LiuZS")
 		(comment 1 "20250613-电池升压改为tps61048，边框形状加入圆角")
 		(comment 2 "20260121-根据原理图重新修改")
+		(comment 3 "20260203-根据原理图重新修改")
 		(comment 9 "1.6mm 板厚 嘉立创 3313叠层")
 	)
@@
 		(fp_text user "*"
 			(at -1.61925 -2.6518 90)
+			(unlocked yes)
 			(layer "F.SilkS")
 			(effects
@@
 		(fp_text user "*"
 			(at -1.61925 -2.6518 90)
-			(unlocked yes)
 			(layer "F.SilkS")
 			(effects
@@
 	(footprint "Jumper:SolderJumper-3_P1.3mm_Bridged12_Pad1.0x1.5mm"
 		(layer "F.Cu")
-		(at 112.086092 126.2)
+		(at 112.086092 126.2 180)
 		(descr "SMD Solder 3-pad Jumper, 1x1.5mm Pads, 0.3mm gap, pads 1-2 bridged with 1 copper strip")
 		(tags "net tie solder jumper bridged")
@@
 		)
 		(property "Value" "SolderJumper_3_Bridged12"
-			(at 0 2 0)
+			(at 0 2.000001 0)
 			(layer "F.Fab")
 			(effects
@@
 		)
 		(property "Datasheet" ""
-			(at 0 0 0)
+			(at 0 0 180)
 			(unlocked yes)
 			(layer "F.Fab")
@@
 		)
 		(property "Description" "3-pole Solder Jumper, pins 1+2 closed/bridged"
-			(at 0 0 0)
+			(at 0 0 180)
 			(unlocked yes)
 			(layer "F.Fab")
@@
 		)
 		(fp_line
-			(start -2.05 -1)
-			(end 2.05 -1)
+			(start 2.05 1)
+			(end -2.05 1)
 			(stroke
 				(width 0.12)
@@
 		)
 		(fp_line
-			(start -2.05 1)
-			(end -2.05 -1)
+			(start 2.05 -1)
+			(end 2.05 1)
 			(stroke
 				(width 0.12)
@@
 		)
 		(fp_line
-			(start -1.6 1.5)
+			(start -1.3 1.2)
 			(end -1 1.5)
 			(stroke
@@
 		)
 		(fp_line
-			(start -1.3 1.2)
+			(start -1.6 1.5)
 			(end -1 1.5)
 			(stroke
@@
 		)
 		(fp_line
-			(start 2.05 -1)
-			(end 2.05 1)
+			(start -2.05 1)
+			(end -2.05 -1)
 			(stroke
 				(width 0.12)
@@
 		)
 		(fp_line
-			(start 2.05 1)
-			(end -2.05 1)
+			(start -2.05 -1)
+			(end 2.05 -1)
 			(stroke
 				(width 0.12)
@@
 		)
 		(fp_line
-			(start -2.3 -1.25)
-			(end -2.3 1.25)
+			(start 2.3 1.25)
+			(end 2.3 -1.25)
 			(stroke
 				(width 0.05)
@@
 		)
 		(fp_line
-			(start -2.3 -1.25)
-			(end 2.3 -1.25)
+			(start 2.3 1.25)
+			(end -2.3 1.25)
 			(stroke
 				(width 0.05)
@@
 		)
 		(fp_line
-			(start 2.3 1.25)
-			(end -2.3 1.25)
+			(start -2.3 -1.25)
+			(end 2.3 -1.25)
 			(stroke
 				(width 0.05)
@@
 		)
 		(fp_line
-			(start 2.3 1.25)
-			(end 2.3 -1.25)
+			(start -2.3 -1.25)
+			(end -2.3 1.25)
 			(stroke
 				(width 0.05)
@@
 		)
 		(pad "1" smd rect
-			(at -1.3 0)
+			(at -1.3 0 180)
 			(size 1 1.5)
 			(layers "F.Cu" "F.Mask")
-			(net 71 "/SHUT_Trig+")
+			(net 73 "/_FLASH_Trig_")
 			(pinfunction "A")
 			(pintype "passive")
 		)
 		(pad "2" smd rect
-			(at 0 0)
+			(at 0 0 180)
 			(size 1 1.5)
 			(layers "F.Cu" "F.Mask")
@@
 		)
 		(pad "3" smd rect
-			(at 1.3 0)
+			(at 1.3 0 180)
 			(size 1 1.5)
 			(layers "F.Cu" "F.Mask")
-			(net 73 "/_FLASH_Trig_")
+			(net 71 "/SHUT_Trig+")
 			(pinfunction "B")
 			(pintype "passive")
@@
 			)
 		)
-		(fp_text user "${REFERENCE}"
-			(at 0 0 0)
+		(fp_text user "*"
+			(at -0.4953 1.4478 0)
 			(unlocked yes)
 			(layer "B.Fab")
@@
 			)
 		)
-		(fp_text user "*"
-			(at -0.4953 1.4478 0)
+		(fp_text user "${REFERENCE}"
+			(at 0 0 0)
 			(unlocked yes)
 			(layer "B.Fab")
